File: pcb/DitherDrive-Tiny.kicad_pcb (KiCad board)
At the start: 2 copper layers, 80.8 x 73.7 mm, 15 parts, among them Q1 IRF540N, U1 R-78E5.0-0.5, U3 INA219AxD, U4 MIC4427

Commit message: fixes
Parts:
- removed D4: 1N53xxB, Diode_THT:D_DO-201_P15.24mm_Horizontal
- moved D2 14.1 mm to (66.5, 153.4), turned to 180 degrees
Connections:
- D2 pad 1: OUT - -> OUT +
- D2 pad 2: Net-(D2-A) -> OUT -
- Q1 pad 2: +24V -> OUT -
- Q1 pad 3: OUT - -> GND
Routing:
- net GND: track 49.8 -> 71.7 mm
- net +24V: track 47.0 -> 32.4 mm
- net Net-(D2-A): track 8.50 -> 0.00 mm
- net Net-(A1-VSYS): track 134.9 -> 139.2 mm
- net Net-(Q1-G): track 53.5 -> 51.0 mm
- net OUT -: track 31.4 -> 33.4 mm
