File: pcb/DitherDrive-Tiny.kicad_sch (KiCad schematic)
At the start: 15 parts, among them Q1 IRF540N, U1 R-78E5.0-0.5, U3 INA219AxD, U4 MIC4427

Commit message: fixes
Parts:
- removed D4: 1N53xxB, Diode_THT:D_DO-201_P15.24mm_Horizontal, symbol Diode:1N53xxB
Connections:
- net +24V: no longer Q1.2 (D)
- net GND: now also Q1.3 (S)
- net OUT +: now also D2.1 (K)
- net OUT -: now also D2.2 (A), Q1.2 (D); no longer D2.1 (K), Q1.3 (S)
Other:
- moved on the sheet: D2, Q1
